File: elpass.kicad_pcb (KiCad board)
At the start: 4 copper layers, 72.4 x 70.2 mm, 218 parts, among them J1 USB_C_Receptacle_USB2.0_16P, J2 HDMI_A, J3 USB_A, J5 Conn_01x04, J6 Conn_02x10_Odd_Even, Q1 AO3400A, Q2 AO3400A, Q3 AO3400A, Q4 SS8050, SW1 TS-1088-AR02016, SW2 TS24CA, U1 TPS563201, U12 ZX-SH1.0-8PLT, U13 TXS0108EPW, U14 TF-123-ARP9H17, U15 TXS0108EPW, U2 CH224K, U3 EA3059, U4 xc7z010clg400, U5 MAX811TEUS-T, U6 XPT2046TS, U7 RL-SM02BD-RTL8723BS, U8 USB3320C-EZK-TR, U9 MT41K256M16TW, X1 3225 50MHz, Y1 24MHz

Commit message: some fixes
Parts:
- removed C4: 1uF, Capacitor_SMD:C_0402_1005Metric
- removed C78, C83: 22pF, Capacitor_SMD:C_0402_1005Metric
- removed J1: USB_C_Receptacle_USB2.0_16P, Connector_USB:USB_C_Receptacle_HRO_TYPE-C-31-M-12
- removed R1: 10K, Resistor_SMD:R_0402_1005Metric
- removed R2: 1K, Resistor_SMD:R_0402_1005Metric
- removed U2: CH224K, EasyEDA:ESSOP-10_L4.9-W3.9-P1.0-LS6.0-TL-EP
- removed Y1: 24MHz, Crystal:Crystal_SMD_3225-4Pin_3.2x2.5mm
- added C75: 470nF, Capacitor_SMD:C_0201_0603Metric, F.Cu at (190.5, 142.1)
- added DC1: DC002-1.3, EasyEDA:DC-IN-TH_DC002-1.3, F.Cu at (201.4, 150.6)
- added R83: 10K, Resistor_SMD:R_0402_1005Metric, B.Cu at (178.6, 90.8)
- added X2: 3225 24MHz, EasyEDA:OSC-SMD_4P-L3.2-W2.5-BL, F.Cu at (192.8, 140.3)
- R12: value 一坨锡 -> 0R
- moved J5 0.31 mm to (198.2, 145.3)
Connections:
- R82 pad 2: /zynq_pl_34/RTL_EN_N -> /zynq_pl_34/RTL_WL_EN_N
- U4 pad T11: unconnected-(U4C-IO_L1P_T0_34-PadT11) -> /zynq_pl_34/RTL_BT_EN_N
- U4 pad U15: /zynq_pl_34/RTL_EN_N -> /zynq_pl_34/RTL_WL_EN_N
- U7 pad 12: /zynq_pl_34/RTL_EN_N -> /zynq_pl_34/RTL_WL_EN_N
- U7 pad 34: /zynq_pl_34/RTL_EN_N -> /zynq_pl_34/RTL_BT_EN_N
- U8 pad 25: Net-(U8-XO) -> unconnected-(U8-XO-Pad25)
Routing:
- net /zynq_pl_34/RTL_EN_N: track 61.1 -> 0.00 mm, vias 2 -> 0
- net /zynq_pl_34/RTL_BT_EN_N: track 0.00 -> 58.6 mm, vias 0 -> 1
- net /zynq_pl_34/RTL_WL_EN_N: track 0.00 -> 46.6 mm, vias 0 -> 2
- net GND: track 308.9 -> 284.5 mm, vias 392 -> 386
- net /Power/PWR_TYPEC_DP: track 17.5 -> 0.00 mm, vias 1 -> 0
- net /Power/PWR_TYPEC_DN: track 17.3 -> 0.00 mm, vias 1 -> 0
- net /Power/PWR_TYPEC_CC1: track 11.1 -> 0.00 mm, vias 1 -> 0
- net /Power/PWR_TYPEC_CC2: track 7.95 -> 0.00 mm, vias 1 -> 0
- net VBUS: track 79.7 -> 73.5 mm, vias 6 -> 5
- net Net-(U8-XO): track 5.67 -> 0.00 mm
- net /Power/CH224_VDD: track 5.21 -> 0.00 mm
- net /zynq_pl_34/ZYNQ_WL_SDIO_D1: track 47.0 -> 50.7 mm
- net +3V3: track 169.5 -> 172.1 mm
- net Net-(U8-REFCLK): track 6.17 -> 3.67 mm
- net Net-(U4C-IO_L3N_T0_DQS_34): track 7.39 -> 4.93 mm
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Other:
- board text added: "elPass V1.1 Shirogane"
- board text removed: "elPass V1 Shirogane"
