File: power.kicad_sch (KiCad schematic)
At the start: 47 parts, among them J1 USB_C_Receptacle_USB2.0_16P, U1 TPS563201, U2 CH224K, U3 EA3059

Commit message: some fixes
Parts:
- removed C4: 1uF, Capacitor_SMD:C_0402_1005Metric, symbol Device:C_Small
- removed J1: USB_C_Receptacle_USB2.0_16P, Connector_USB:USB_C_Receptacle_HRO_TYPE-C-31-M-12, symbol Connector:USB_C_Receptacle_USB2.0_16P
- removed R1: 10K, Resistor_SMD:R_0402_1005Metric, symbol Device:R_Small
- removed R2: 1K, Resistor_SMD:R_0402_1005Metric, symbol Device:R_Small
- removed U2: CH224K, EasyEDA:ESSOP-10_L4.9-W3.9-P1.0-LS6.0-TL-EP, symbol EasyEDA:CH224K
- added DC1: DC002-1.3, EasyEDA:DC-IN-TH_DC002-1.3, symbol EasyEDA:DC002-1.3
Connections:
- net GND: now also DC1.3
- net VBUS: now also DC1.1
- no-connect marks 5 -> 3
Other:
- note removed: "CH224 Configured to trigger 12V"
