File: zynq_pl_34.kicad_sch (KiCad schematic)
At the start: 28 parts, among them J6 Conn_02x10_Odd_Even, Q4 SS8050, U13 TXS0108EPW, U15 TXS0108EPW, U4 xc7z010clg400, U7 RL-SM02BD-RTL8723BS

Commit message: some fixes
Parts:
- added R83: 10K, Resistor_SMD:R_0402_1005Metric, symbol Device:R_Small
Connections:
- net GND: now also R83.1
- net RTL_BT_EN_N: now reaches U4.T11 (IO_L1P_T0_34)
- net RTL_BT_EN_N: now also U7.34 (BT_DIS#), R83.2
- net RTL_EN_N renamed RTL_WL_EN_N
- net RTL_WL_EN_N: no longer U7.34 (BT_DIS#)
- no-connect marks 32 -> 31
Other:
- moved on the sheet: R82
