File: zynq_ps_peri.kicad_sch (KiCad schematic)
At the start: 20 parts, among them J3 USB_A, U14 TF-123-ARP9H17, U4 xc7z010clg400, U8 USB3320C-EZK-TR, Y1 24MHz

Commit message: some fixes
Parts:
- removed C78, C83: 22pF, Capacitor_SMD:C_0402_1005Metric, symbol Device:C_Small
- removed Y1: 24MHz, Crystal:Crystal_SMD_3225-4Pin_3.2x2.5mm, symbol Device:Crystal_GND24
- added C75: 470nF, Capacitor_SMD:C_0201_0603Metric, symbol Device:C_Small
- added X2: 3225 24MHz, EasyEDA:OSC-SMD_4P-L3.2-W2.5-BL, symbol EasyEDA:OT322550MJBA4SL
Connections:
- net +3V3: now also C75.1, X2.4 (VDD)
- net GND: now also C75.2, X2.2 (GND)
- net at U8.26 (REFCLK): now also X2.3 (OUTPUT)
- no-connect marks 27 -> 29
